File: mechanical/Circuit/PiRCS2Updater/PiRCS2Updater-simple.kicad_sch (KiCad schematic)
At the start: 18 parts, among them J1 USB_B_Micro, J10 Conn_01x01, J11 Charger USB C, J2 USB Data, J3 Power In, J4 Conn_01x02, J5 RC-2 USB C, J6 Battery, J7 Battery, J8 Switch, J9 Conn_01x02, SW1 SW_DPST_x2

Commit message: V3.0.0c circuit ans 3dprint updates
Parts:
- J1: value USB_B_Micro -> Charge plug
- J11: value Charger USB C -> Charger in
- J5: value RC-2 USB C -> USB C
Connections:
- net 5V: now also J5.A4 (VBUS), J5.A9 (VBUS), J5.B4 (VBUS), J5.B9 (VBUS), R2.1, R5.1
- net at R2.2: now also J5.B5 (CC2); no longer J5.A5 (CC1)
- net at R5.2: now also J5.A5 (CC1); no longer J5.B5 (CC2)
- now unconnected: J2.1 (VBUS)
Other:
- note added: "CC1, CC2: 56k to 5V = we are a USB source"
- note added: "RC-2 VBUS = 5V (always on)"
- note added: "SW1 closed grounds EN = OFF, open = ON"
- note removed: "Closed is OFF"
- note removed: "GPIO4"
- note removed: "V3.3"
- moved on the sheet: J5, R2, R4, R5
