File: mechanical/Circuit/PiRCS2Updater/xPiRCS2Updater.kicad_sch (KiCad schematic)
At the start: 18 parts, among them J1 USB_B_Micro, J10 Conn_01x01, J11 Charger USB C, J2 USB Data, J3 Power In, J4 Conn_01x02, J5 RC-2 USB C, J6 Battery, J7 Battery, J8 Switch, J9 Conn_01x02, SW1 SW_DPST_x2

Commit message: V3.0.0c circuit ans 3dprint updates
Parts:
- removed J11: Charger USB C, symbol Connector:USB_B_Micro
- added D4, D5: 1N4148, Diode_THT:D_DO-35_SOD27_P7.62mm_Horizontal, symbol Diode:1N4148
- added Q1, Q2: IRLML6402, Package_TO_SOT_SMD:SOT-23, symbol Transistor_FET:IRLML6402
- added R1: 1M, symbol Device:R
- J5: value RC-2 USB C -> USB C
Connections:
- net at J5.A4 (VBUS), J5.A9 (VBUS), J5.B4 (VBUS)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: now also J1.1 (VBUS), Q1.3 (D); no longer J2.1 (VBUS), R2.1, R5.1
- net at R2.2: now also J5.B5 (CC2), D5.1 (K); no longer J5.A5 (CC1)
- net at D3.2 (A), R4.2: now also J9.7 (GPIO_4)
- net at R5.2: now also J5.A5 (CC1), D4.1 (K); no longer J5.B5 (CC2)
- net 5V: no longer names the net of D2.2 (A), J3.1 (VBUS), J4.2 (Pin_2)
- net GND: no longer names the net of J1.5 (GND), J2.4 (ID), J2.5 (GND), J5.A1 (GND), J5.A12 (GND), J5.B1 (GND), J5.B12 (GND)
- net GND: no longer J3.5 (GND), J4.1 (Pin_1), R3.2
- new net: D4.2 (A), D5.2 (A), Q1.1 (G), Q2.1 (G), R1.1
- new net: Q1.2 (S), Q2.2 (S), R1.2, R2.1, R5.1
- new net: J3.5 (GND), J4.1 (Pin_1), R3.2
Other:
- note added: "Open is ON"
- note added: "VBUS"
- note removed: "Closed is OFF"
- note removed: "GPIO4"
- note removed: "V3.3"
- moved on the sheet: J5, R2, R4, R5
